Commit message: Added teleoperation_camera node (has to fine tune transforms)

File: robot_moveit/config/robot_one.ros2_control.xacro (robot description, xacro)
@@ -99,11 +99,4 @@
                 <state_interface name="velocity"/>
             </joint>
-            <joint name="right_gripper_joint_robot_1">
-                <command_interface name="position"/>
-                <state_interface name="position">
-                  <param name="initial_value">${initial_positions['right_gripper_joint_robot_1']}</param>
-                </state_interface>
-                <state_interface name="velocity"/>
-            </joint>
             <joint name="left_gripper_joint_robot_2">
                 <command_interface name="position"/>
@@ -113,11 +106,4 @@
                 <state_interface name="velocity"/>
             </joint>
-            <joint name="right_gripper_joint_robot_2">
-                <command_interface name="position"/>
-                <state_interface name="position">
-                  <param name="initial_value">${initial_positions['right_gripper_joint_robot_2']}</param>
-                </state_interface>
-                <state_interface name="velocity"/>
-            </joint>
         </ros2_control>
     </xacro:macro>

File: sereact/src/description/robot.urdf.xacro (robot description, xacro)
@@ -224,4 +224,5 @@
     <axis xyz="-1 0 0"/>
     <limit effort="10" velocity="1.0" lower="0.0" upper="0.06"/>
+    <mimic joint="left_gripper_joint_robot_1" multiplier="1" offset="0"/>
   </joint>
   <!-- ========== right robot ========== -->
@@ -436,4 +437,5 @@
     <axis xyz="-1 0 0"/>
     <limit effort="10" velocity="1.0" lower="0.0" upper="0.06"/>
+    <mimic joint="left_gripper_joint_robot_2" multiplier="1" offset="0"/>
   </joint>
 </robot>
