Commit message: Modified moveit configuration and added arguments to imitation algorithm

File: robot_moveit/config/dual_arm_robot.ros2_control.xacro (robot description, xacro)
@@ -1,5 +1,5 @@
 <?xml version="1.0"?>
 <robot xmlns:xacro="http://www.ros.org/wiki/xacro">
-    <xacro:macro name="robot_one_ros2_control" params="name initial_positions_file">
+    <xacro:macro name="dual_arm_robot_ros2_control" params="name initial_positions_file">
         <xacro:property name="initial_positions" value="${xacro.load_yaml(initial_positions_file)['initial_positions']}"/>
         <ros2_control name="${name}" type="system">

File: sereact/src/description/robot.urdf.xacro (robot description, xacro)
@@ -1,4 +1,4 @@
 <?xml version="1.0"?>
-<robot name="robot_one" xmlns:xacro="http://www.ros.org/wiki/xacro">
+<robot name="dual_arm_robot" xmlns:xacro="http://www.ros.org/wiki/xacro">
     <!-- ========== BASE LINK ========== -->
   <link name="base_link">
@@ -10,8 +10,15 @@
     <collision>
       <origin xyz="0 0 0.1" rpy="0 0 0"/>
-      <geometry><box size="3.0 1.5 0.05"/></geometry>
+      <geometry><box size="3.0 3.0 0.05"/></geometry>
     </collision>
   </link>
   <!-- ========== left robot ========== -->
+    <link name="base_link_robot_1"></link>
+    <joint name="basejoint_robot_1" type="fixed">
+      <parent link="base_link"/>
+      <child link="base_link_robot_1"/>
+      <origin xyz="0 -0.75 0.1" rpy="0 0 0"/>
+      <axis xyz="0 0 1"/>
+    </joint>
   <!-- ========== JOINT 1 ========== -->
   <link name="link1_robot_1">
@@ -32,7 +39,7 @@
   </link>
   <joint name="joint1_robot_1" type="revolute">
-    <parent link="base_link"/>
+    <parent link="base_link_robot_1"/>
     <child link="link1_robot_1"/>
-    <origin xyz="0 -0.75 0.1" rpy="0 0 0"/>
+    <origin xyz="0 0 0" rpy="0 0 0"/>
     <axis xyz="0 0 1"/>
     <limit effort="10" velocity="10" lower="-3.14" upper="3.14"/>
@@ -227,4 +234,11 @@
   </joint>
   <!-- ========== right robot ========== -->
+    <link name="base_link_robot_2"></link>
+    <joint name="basejoint_robot_2" type="fixed">
+      <parent link="base_link"/>
+      <child link="base_link_robot_2"/>
+      <origin xyz="0 0.75 0.1" rpy="0 0 0"/>
+      <axis xyz="0 0 1"/>
+    </joint>
   <!-- ========== JOINT 1 ========== -->
   <link name="link1_robot_2">
@@ -245,7 +259,7 @@
   </link>
   <joint name="joint1_robot_2" type="revolute">
-    <parent link="base_link"/>
+    <parent link="base_link_robot_2"/>
     <child link="link1_robot_2"/>
-    <origin xyz="0 0.75 0.1" rpy="0 0 0"/>
+    <origin xyz="0 0 0" rpy="0 0 0"/>
     <axis xyz="0 0 1"/>
     <limit effort="10" velocity="1.0" lower="-3.14" upper="3.14"/>
