Commit message: Adjusted robots configurations

File: robot_main/src/description/robot.urdf.xacro (robot description, xacro)
@@ -114,5 +114,10 @@
     <child link="link4_robot_1"/>
     <origin xyz="0 0 0.19" rpy="0 0 0"/>
-    <axis xyz="0 1 0"/>
+    <!-- PATCH: was "0 1 0". With axes z,y,y,y,y,z the arm only spans a 5-D pose
+         manifold (position and tool axis always coplanar with the base z-axis),
+         so full 6D IK goals are unsolvable. Making joint4 a forearm roll (z)
+         yields a z,y,y,z,y,z structure: articulated arm + roll-pitch-roll wrist,
+         a proper 6-DOF manipulator. -->
+    <axis xyz="0 0 1"/>
     <limit effort="10" velocity="1.0" lower="-3.14" upper="3.14"/>
   </joint>
@@ -230,4 +235,8 @@
     <origin xyz="0.067 0 0.02" rpy="0 0 0"/>
     <axis xyz="-1 0 0"/>
+    <!-- PATCH: right finger mirrors the left one. Combined with the mimic entry in
+         the ros2_control xacro, this puts the joint in /joint_states so its TF
+         exists and MoveIt stops warning about an incomplete robot state. -->
+    <mimic joint="left_gripper_joint_robot_1" multiplier="1.0" offset="0.0"/>
     <limit effort="10" velocity="1.0" lower="0.0" upper="0.06"/>
     <mimic joint="left_gripper_joint_robot_1" multiplier="1" offset="0"/>
@@ -334,5 +343,6 @@
     <child link="link4_robot_2"/>
     <origin xyz="0 0 0.19" rpy="0 0 0"/>
-    <axis xyz="0 1 0"/>
+    <!-- PATCH: was "0 1 0" (see joint4_robot_1 for rationale) -->
+    <axis xyz="0 0 1"/>
     <limit effort="10" velocity="1.0" lower="-2.0" upper="2.0"/>
   </joint>
@@ -450,4 +460,8 @@
     <origin xyz="0.067 0 0.02" rpy="0 0 0"/>
     <axis xyz="-1 0 0"/>
+    <!-- PATCH: right finger mirrors the left one. Combined with the mimic entry in
+         the ros2_control xacro, this puts the joint in /joint_states so its TF
+         exists and MoveIt stops warning about an incomplete robot state. -->
+    <mimic joint="left_gripper_joint_robot_2" multiplier="1.0" offset="0.0"/>
     <limit effort="10" velocity="1.0" lower="0.0" upper="0.06"/>
     <mimic joint="left_gripper_joint_robot_2" multiplier="1" offset="0"/>

File: robot_moveit/config/config/dual_arm_robot.ros2_control.xacro (robot description, xacro)
@@ -106,4 +106,23 @@
                 <state_interface name="velocity"/>
             </joint>
+            <!-- PATCH: right fingers as mimic joints so the
+                 joint_state_broadcaster publishes them (valid TF for the right
+                 finger links, no MoveIt incomplete-state warnings).
+                 The mimic relationship itself lives in the URDF <mimic> tag on
+                 these joints; ros2_control (Iron/Jazzy and newer) parses that
+                 tag directly and REQUIRES activated mimic joints to have no
+                 command interfaces - state interfaces only. mock hardware then
+                 fills their position/velocity from the mimicked joint.
+                 (On Humble only, mimic was configured here instead, via
+                 <param name="mimic">left_gripper_joint_robot_N</param> and
+                 <param name="multiplier">1</param>.) -->
+            <joint name="right_gripper_joint_robot_1">
+                <state_interface name="position"/>
+                <state_interface name="velocity"/>
+            </joint>
+            <joint name="right_gripper_joint_robot_2">
+                <state_interface name="position"/>
+                <state_interface name="velocity"/>
+            </joint>
         </ros2_control>
     </xacro:macro>
